File: rom-dumper/pps-rom-dumper/inputs.sch (KiCad schematic (older format))
At the start: 16 parts

Commit message: Updates
Parts:
- R14, R16, R18, R20, R22, R24, R26, R28: value 4M -> 47k
- R15, R17, R19, R21, R23, R25, R27, R29: value 1M -> 10k
Changed lines of the file:
@@
 AR Path="/641D5056/641D56EA" Ref="R20"  Part="1"
 F 0 "R20" H 1909 1196 50  0000 L CNN
-F 1 "4M" H 1909 1105 50  0000 L CNN
+F 1 "47k" H 1909 1105 50  0000 L CNN
 F 2 "Resistor_SMD:R_0805_2012Metric_Pad1.20x1.40mm_HandSolder" H 1850 1150 50  0001 C CNN
 F 3 "~" H 1850 1150 50  0001 C CNN
@@
 AR Path="/641D5056/641D56F0" Ref="R21"  Part="1"
 F 0 "R21" H 1909 1521 50  0000 L CNN
-F 1 "1M" H 1909 1430 50  0000 L CNN
+F 1 "10k" H 1909 1430 50  0000 L CNN
 F 2 "Resistor_SMD:R_0805_2012Metric_Pad1.20x1.40mm_HandSolder" H 1850 1475 50  0001 C CNN
 F 3 "~" H 1850 1475 50  0001 C CNN
@@
 AR Path="/641D5056/641D5D99" Ref="R16"  Part="1"
 F 0 "R16" H 1834 2271 50  0000 L CNN
-F 1 "4M" H 1834 2180 50  0000 L CNN
+F 1 "47k" H 1834 2180 50  0000 L CNN
 F 2 "Resistor_SMD:R_0805_2012Metric_Pad1.20x1.40mm_HandSolder" H 1775 2225 50  0001 C CNN
 F 3 "~" H 1775 2225 50  0001 C CNN
@@
 AR Path="/641D5056/641D5D9F" Ref="R17"  Part="1"
 F 0 "R17" H 1834 2596 50  0000 L CNN
-F 1 "1M" H 1834 2505 50  0000 L CNN
+F 1 "10k" H 1834 2505 50  0000 L CNN
 F 2 "Resistor_SMD:R_0805_2012Metric_Pad1.20x1.40mm_HandSolder" H 1775 2550 50  0001 C CNN
 F 3 "~" H 1775 2550 50  0001 C CNN
@@
 AR Path="/641D5056/641D664B" Ref="R14"  Part="1"
 F 0 "R14" H 1809 3521 50  0000 L CNN
-F 1 "4M" H 1809 3430 50  0000 L CNN
+F 1 "47k" H 1809 3430 50  0000 L CNN
 F 2 "Resistor_SMD:R_0805_2012Metric_Pad1.20x1.40mm_HandSolder" H 1750 3475 50  0001 C CNN
 F 3 "~" H 1750 3475 50  0001 C CNN
@@
 AR Path="/641D5056/641D6651" Ref="R15"  Part="1"
 F 0 "R15" H 1809 3846 50  0000 L CNN
-F 1 "1M" H 1809 3755 50  0000 L CNN
+F 1 "10k" H 1809 3755 50  0000 L CNN
 F 2 "Resistor_SMD:R_0805_2012Metric_Pad1.20x1.40mm_HandSolder" H 1750 3800 50  0001 C CNN
 F 3 "~" H 1750 3800 50  0001 C CNN
@@
 AR Path="/641D5056/641D6C9B" Ref="R18"  Part="1"
 F 0 "R18" H 1859 4746 50  0000 L CNN
-F 1 "4M" H 1859 4655 50  0000 L CNN
+F 1 "47k" H 1859 4655 50  0000 L CNN
 F 2 "Resistor_SMD:R_0805_2012Metric_Pad1.20x1.40mm_HandSolder" H 1800 4700 50  0001 C CNN
 F 3 "~" H 1800 4700 50  0001 C CNN
@@
 AR Path="/641D5056/641D6CA1" Ref="R19"  Part="1"
 F 0 "R19" H 1859 5071 50  0000 L CNN
-F 1 "1M" H 1859 4980 50  0000 L CNN
+F 1 "10k" H 1859 4980 50  0000 L CNN
 F 2 "Resistor_SMD:R_0805_2012Metric_Pad1.20x1.40mm_HandSolder" H 1800 5025 50  0001 C CNN
 F 3 "~" H 1800 5025 50  0001 C CNN
@@
 AR Path="/641D5056/641D7480" Ref="R28"  Part="1"
 F 0 "R28" H 3984 1271 50  0000 L CNN
-F 1 "4M" H 3984 1180 50  0000 L CNN
+F 1 "47k" H 3984 1180 50  0000 L CNN
 F 2 "Resistor_SMD:R_0805_2012Metric_Pad1.20x1.40mm_HandSolder" H 3925 1225 50  0001 C CNN
 F 3 "~" H 3925 1225 50  0001 C CNN
@@
 AR Path="/641D5056/641D7486" Ref="R29"  Part="1"
 F 0 "R29" H 3984 1596 50  0000 L CNN
-F 1 "1M" H 3984 1505 50  0000 L CNN
+F 1 "10k" H 3984 1505 50  0000 L CNN
 F 2 "Resistor_SMD:R_0805_2012Metric_Pad1.20x1.40mm_HandSolder" H 3925 1550 50  0001 C CNN
 F 3 "~" H 3925 1550 50  0001 C CNN
@@
 AR Path="/641D5056/641D7FFB" Ref="R26"  Part="1"
 F 0 "R26" H 3959 2446 50  0000 L CNN
-F 1 "4M" H 3959 2355 50  0000 L CNN
+F 1 "47k" H 3959 2355 50  0000 L CNN
 F 2 "Resistor_SMD:R_0805_2012Metric_Pad1.20x1.40mm_HandSolder" H 3900 2400 50  0001 C CNN
 F 3 "~" H 3900 2400 50  0001 C CNN
@@
 AR Path="/641D5056/641D8001" Ref="R27"  Part="1"
 F 0 "R27" H 3959 2771 50  0000 L CNN
-F 1 "1M" H 3959 2680 50  0000 L CNN
+F 1 "10k" H 3959 2680 50  0000 L CNN
 F 2 "Resistor_SMD:R_0805_2012Metric_Pad1.20x1.40mm_HandSolder" H 3900 2725 50  0001 C CNN
 F 3 "~" H 3900 2725 50  0001 C CNN
@@
 AR Path="/641D5056/641D8D08" Ref="R24"  Part="1"
 F 0 "R24" H 3884 3496 50  0000 L CNN
-F 1 "4M" H 3884 3405 50  0000 L CNN
+F 1 "47k" H 3884 3405 50  0000 L CNN
 F 2 "Resistor_SMD:R_0805_2012Metric_Pad1.20x1.40mm_HandSolder" H 3825 3450 50  0001 C CNN
 F 3 "~" H 3825 3450 50  0001 C CNN
@@
 AR Path="/641D5056/641D8D0E" Ref="R25"  Part="1"
 F 0 "R25" H 3884 3821 50  0000 L CNN
-F 1 "1M" H 3884 3730 50  0000 L CNN
+F 1 "10k" H 3884 3730 50  0000 L CNN
 F 2 "Resistor_SMD:R_0805_2012Metric_Pad1.20x1.40mm_HandSolder" H 3825 3775 50  0001 C CNN
 F 3 "~" H 3825 3775 50  0001 C CNN
@@
 AR Path="/641D5056/641D9AD7" Ref="R22"  Part="1"
 F 0 "R22" H 3859 4671 50  0000 L CNN
-F 1 "4M" H 3859 4580 50  0000 L CNN
+F 1 "47k" H 3859 4580 50  0000 L CNN
 F 2 "Resistor_SMD:R_0805_2012Metric_Pad1.20x1.40mm_HandSolder" H 3800 4625 50  0001 C CNN
 F 3 "~" H 3800 4625 50  0001 C CNN
@@
 AR Path="/641D5056/641D9ADD" Ref="R23"  Part="1"
 F 0 "R23" H 3859 4996 50  0000 L CNN
-F 1 "1M" H 3859 4905 50  0000 L CNN
+F 1 "10k" H 3859 4905 50  0000 L CNN
 F 2 "Resistor_SMD:R_0805_2012Metric_Pad1.20x1.40mm_HandSolder" H 3800 4950 50  0001 C CNN
 F 3 "~" H 3800 4950 50  0001 C CNN
