File: rom-dumper/pps-rom-dumper/pps-rom-dumper.kicad_pcb (KiCad board)
At the start: 2 copper layers, 96.5 x 61 mm, 67 parts, among them J1 Conn_01x03_Female, U1 Pico, U2 pps4-rom-a05, U3 Regulator_Switching_MT3608

Commit message: Updates
Parts:
- C5, C6: value C_Small -> 100nF
- R14, R16, R18, R20, R22, R24, R26, R28: value 4M -> 47k
- R15, R17, R19, R21, R23, R25, R27, R29: value 1M -> 10k
- R34: value 100k -> 47k
- R35: value 5k -> 220
- R36: value 1k -> 1500
Changed lines of the file:
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@@
   )
   (setup
-    (last_trace_width 0.4)
+    (last_trace_width 0.25)
     (user_trace_width 0.4)
     (user_trace_width 1)
@@
     (add_net "Net-(U1-Pad37)")
     (add_net "Net-(U1-Pad40)")
+    (add_net "Net-(U2-Pad10)")
+    (add_net "Net-(U2-Pad14)")
+    (add_net "Net-(U2-Pad17)")
+    (add_net "Net-(U2-Pad18)")
+    (add_net "Net-(U2-Pad20)")
+    (add_net "Net-(U2-Pad23)")
+    (add_net "Net-(U2-Pad25)")
+    (add_net "Net-(U2-Pad38)")
+    (add_net "Net-(U2-Pad40)")
+    (add_net "Net-(U2-Pad5)")
+    (add_net "Net-(U3-Pad6)")
     (add_net PA11X)
     (add_net PAB1)
@@
       (effects (font (size 1 1) (thickness 0.15)))
     )
-    (fp_text value C_Small (at 0 2.3) (layer F.Fab)
+    (fp_text value 100nF (at 0 2.3) (layer F.Fab)
       (effects (font (size 1 1) (thickness 0.15)))
     )
@@
       (effects (font (size 1 1) (thickness 0.15)))
     )
-    (fp_text value C_Small (at 0 2.3) (layer F.Fab)
+    (fp_text value 100nF (at 0 2.3) (layer F.Fab)
       (effects (font (size 1 1) (thickness 0.15)))
     )
@@
       (effects (font (size 1 1) (thickness 0.15)))
     )
-    (fp_text value 1k (at 0 1.65) (layer F.Fab)
+    (fp_text value 1500 (at 0 1.65) (layer F.Fab)
       (effects (font (size 1 1) (thickness 0.15)))
     )
@@
       (effects (font (size 1 1) (thickness 0.15)))
     )
-    (fp_text value 5k (at 0 1.65 90) (layer F.Fab)
+    (fp_text value 220 (at 0 1.65 90) (layer F.Fab)
       (effects (font (size 1 1) (thickness 0.15)))
     )
@@
       (effects (font (size 1 1) (thickness 0.15)))
     )
-    (fp_text value 100k (at 0 1.65 90) (layer F.Fab)
+    (fp_text value 47k (at 0 1.65 90) (layer F.Fab)
       (effects (font (size 1 1) (thickness 0.15)))
     )
@@
       (effects (font (size 1 1) (thickness 0.15)))
     )
-    (fp_text value 1M (at 0 1.65) (layer F.Fab)
+    (fp_text value 10k (at 0 1.65) (layer F.Fab)
       (effects (font (size 1 1) (thickness 0.15)))
     )
@@
       (effects (font (size 1 1) (thickness 0.15)))
     )
-    (fp_text value 4M (at 0 1.65) (layer F.Fab)
+    (fp_text value 47k (at 0 1.65) (layer F.Fab)
       (effects (font (size 1 1) (thickness 0.15)))
     )
@@
       (effects (font (size 1 1) (thickness 0.15)) (justify mirror))
     )
-    (fp_text value 1M (at 0 -1.65) (layer B.Fab)
+    (fp_text value 10k (at 0 -1.65) (layer B.Fab)
       (effects (font (size 1 1) (thickness 0.15)) (justify mirror))
     )
@@
       (effects (font (size 1 1) (thickness 0.15)) (justify mirror))
     )
-    (fp_text value 4M (at 0 -1.65) (layer B.Fab)
+    (fp_text value 47k (at 0 -1.65) (layer B.Fab)
       (effects (font (size 1 1) (thickness 0.15)) (justify mirror))
     )
@@
       (effects (font (size 1 1) (thickness 0.15)))
     )
-    (fp_text value 1M (at 0 1.65) (layer F.Fab)
+    (fp_text value 10k (at 0 1.65) (layer F.Fab)
       (effects (font (size 1 1) (thickness 0.15)))
     )
@@
       (effects (font (size 1 1) (thickness 0.15)))
     )
-    (fp_text value 4M (at 0 1.65) (layer F.Fab)
+    (fp_text value 47k (at 0 1.65) (layer F.Fab)
       (effects (font (size 1 1) (thickness 0.15)))
     )
@@
       (effects (font (size 1 1) (thickness 0.15)) (justify mirror))
     )
-    (fp_text value 1M (at 0 -1.65) (layer B.Fab)
+    (fp_text value 10k (at 0 -1.65) (layer B.Fab)
       (effects (font (size 1 1) (thickness 0.15)) (justify mirror))
     )
@@
       (effects (font (size 1 1) (thickness 0.15)) (justify mirror))
     )
-    (fp_text value 4M (at 0 -1.65) (layer B.Fab)
+    (fp_text value 47k (at 0 -1.65) (layer B.Fab)
       (effects (font (size 1 1) (thickness 0.15)) (justify mirror))
     )
@@
       (effects (font (size 1 1) (thickness 0.15)) (justify mirror))
     )
-    (fp_text value 1M (at 0 -1.65) (layer B.Fab)
+    (fp_text value 10k (at 0 -1.65) (layer B.Fab)
       (effects (font (size 1 1) (thickness 0.15)) (justify mirror))
     )
@@
       (effects (font (size 1 1) (thickness 0.15)) (justify mirror))
     )
-    (fp_text value 4M (at 0 -1.65) (layer B.Fab)
+    (fp_text value 47k (at 0 -1.65) (layer B.Fab)
       (effects (font (size 1 1) (thickness 0.15)) (justify mirror))
     )
@@
       (effects (font (size 1 1) (thickness 0.15)))
     )
-    (fp_text value 1M (at 0 1.65) (layer F.Fab)
+    (fp_text value 10k (at 0 1.65) (layer F.Fab)
       (effects (font (size 1 1) (thickness 0.15)))
     )
@@
       (effects (font (size 1 1) (thickness 0.15)))
     )
-    (fp_text value 4M (at 0 1.65) (layer F.Fab)
+    (fp_text value 47k (at 0 1.65) (layer F.Fab)
       (effects (font (size 1 1) (thickness 0.15)))
     )
@@
       (effects (font (size 1 1) (thickness 0.15)))
     )
-    (fp_text value 1M (at 0 1.65) (layer F.Fab)
+    (fp_text value 10k (at 0 1.65) (layer F.Fab)
       (effects (font (size 1 1) (thickness 0.15)))
     )
@@
       (effects (font (size 1 1) (thickness 0.15)))
     )
-    (fp_text value 4M (at 0 1.65) (layer F.Fab)
+    (fp_text value 47k (at 0 1.65) (layer F.Fab)
       (effects (font (size 1 1) (thickness 0.15)))
     )
@@
       (effects (font (size 1 1) (thickness 0.15)) (justify mirror))
     )
-    (fp_text value 1M (at 0 -1.65) (layer B.Fab)
+    (fp_text value 10k (at 0 -1.65) (layer B.Fab)
       (effects (font (size 1 1) (thickness 0.15)) (justify mirror))
     )
@@
       (effects (font (size 1 1) (thickness 0.15)) (justify mirror))
     )
-    (fp_text value 4M (at 0 -1.65) (layer B.Fab)
+    (fp_text value 47k (at 0 -1.65) (layer B.Fab)
       (effects (font (size 1 1) (thickness 0.15)) (justify mirror))
     )
