File: rom-dumper/pps-rom-dumper/pps-rom-dumper.sch (KiCad schematic (older format))
At the start: 4 parts

Commit message: Updates
Parts:
- removed U? (x2): New_Library_MAX6921AWI, Package_SO:SOIC-28W_7.5x17.9mm_P1.27mm, symbol cq1re1-cache:New_Library_MAX6921AWI
- added C1, C2: 22uF, Capacitor_SMD:C_1210_3225Metric_Pad1.33x2.70mm_HandSolder, symbol Device:C_Small
- added C3: 10uF, Capacitor_SMD:C_1210_3225Metric_Pad1.33x2.70mm_HandSolder, symbol Device:C_Small
- added C4: 100nF, Capacitor_SMD:C_1210_3225Metric_Pad1.33x2.70mm_HandSolder, symbol Device:C_Small
- added C5, C6: C_Small, Capacitor_SMD:C_1210_3225Metric_Pad1.33x2.70mm_HandSolder, symbol Device:C_Small
- added D1: SS36, Diode_SMD:D_SOD-123, symbol Device:D
- added J1: Conn_01x03_Female, Connector_PinHeader_2.54mm:PinHeader_1x03_P2.54mm_Vertical, symbol Connector:Conn_01x03_Female
- added JP1: Jumper_NO_Small, psion_org_2:SolderJumper-2_P1.3mm_Open_Pad0.8x0.8mm, symbol Device:Jumper_NO_Small
- added JP2: SolderJumper_2_Open, psion_org_2:SolderJumper-2_P1.3mm_Open_Pad0.8x0.8mm, symbol Jumper:SolderJumper_2_Open
- added L1: 22uH, Inductor_SMD:L_Coilcraft_LPS5030, symbol pspice:INDUCTOR
- added R34: 100k, Resistor_SMD:R_0805_2012Metric, symbol Device:R_Small
- added R35: 5k, Resistor_SMD:R_0805_2012Metric, symbol Device:R_Small
- added R36: 1k, Resistor_SMD:R_0805_2012Metric, symbol Device:R_Small
- added U3: Regulator_Switching_MT3608, Package_TO_SOT_SMD:SOT-23-6, symbol cq1re1-cache:Regulator_Switching_MT3608
- U1: renamed from U?; footprint RPi_Pico:RPi_Pico_SMD_TH -> rp2040:RPi_Pico_SMD_TH
- U2: renamed from U?; footprint (none) -> ajm_kicad:qip42
Connections:
- net VDD: now also U1.13 (GND), U1.18 (GND), U1.23 (GND), U1.28 (GND), U1.3 (GND), U1.38 (GND), U1.42 (GND), U1.8 (GND), C1.2, C2.2, C3.2, C4.2, C5.2, C6.2, J1.2 (Pin_2), R36.2, U3.2 (GND)
- net VSS: now also C3.1, C4.1, C5.1, C6.1, JP2.2 (B)
- net IP_ID1: now reaches U1.1 (GPIO0)
- net IP_ID8: now reaches U1.10 (GPIO7)
- net PAB1: now reaches U1.11 (GPIO8)
- net PAB2: now reaches U1.12 (GPIO9)
- net PAB3: now reaches U1.14 (GPIO10)
- net PAB4: now reaches U1.15 (GPIO11)
- net PAB5: now reaches U1.16 (GPIO12)
- net PAB6: now reaches U1.17 (GPIO13)
- net PAB7: now reaches U1.19 (GPIO14)
- net IP_ID2: now reaches U1.2 (GPIO1)
- net PAB8: now reaches U1.20 (GPIO15)
- net PAB9: now reaches U1.21 (GPIO16)
- net PAB10: now reaches U1.22 (GPIO17)
- net PA11X: now reaches U1.24 (GPIO18)
- net PCLKB: now reaches U1.25 (GPIO19)
- net PCLKA: now reaches U1.26 (GPIO20)
- net PAS1: now reaches U1.27 (GPIO21)
- net PAS2: now reaches U1.29 (GPIO22)
- net PAS3: now reaches U1.31 (GPIO26_ADC0)
- net PAS4: now reaches U1.32 (GPIO27_ADC1)
- net VSYS: now reaches U1.39 (VSYS)
- net VSYS: now also JP1.1
- net IP_ID3: now reaches U1.4 (GPIO2)
- net SWCLK: now reaches U1.41 (SWCLK)
- net SWCLK: now also J1.3 (Pin_3)
- net SWD: now reaches U1.43 (SWDIO)
- net SWD: now also J1.1 (Pin_1)
- net IP_ID4: now reaches U1.5 (GPIO3)
- net IP_ID5: now reaches U1.6 (GPIO4)
- net IP_ID6: now reaches U1.7 (GPIO5)
- net IP_ID7: now reaches U1.9 (GPIO6)
- new net: R34.2, R35.1, U3.3 (FB)
- new net: R35.2, R36.1
- new net: C1.1, JP1.2, L1.1, U3.4 (EN), U3.5 (IN)
- new net: C2.1, D1.1 (K), JP2.1 (A), R34.1
- new net: D1.2 (A), L1.2, U3.1 (SW)
Other:
- note added: "Check values\n"
- note added: "JP1: leave open until output of U3 is confirmed\nat 10.5V"
- moved on the sheet: U1, U2

Commit message: Updates
Parts:
- C5, C6: value C_Small -> 100nF
- R34: value 100k -> 47k
- R35: value 5k -> 220
- R36: value 1k -> 1500
Other:
- note added: "JP1: leave open until output of U3 is confirmed\nat 17V"
- note removed: "JP1: leave open until output of U3 is confirmed\nat 10.5V"
Changed lines of the file:
@@
 AR Path="/630E4C46/641A8E81" Ref="R?"  Part="1"
 F 0 "R35" H 4209 2596 50  0000 L CNN
-F 1 "5k" H 4209 2505 50  0000 L CNN
+F 1 "220" H 4209 2505 50  0000 L CNN
 F 2 "Resistor_SMD:R_0805_2012Metric" H 4150 2550 50  0001 C CNN
 F 3 "~" H 4150 2550 50  0001 C CNN
@@
 AR Path="/630E4C46/641A8EA5" Ref="R?"  Part="1"
 F 0 "R34" H 4209 2146 50  0000 L CNN
-F 1 "100k" H 4209 2055 50  0000 L CNN
+F 1 "47k" H 4209 2055 50  0000 L CNN
 F 2 "Resistor_SMD:R_0805_2012Metric" H 4150 2100 50  0001 C CNN
 F 3 "~" H 4150 2100 50  0001 C CNN
@@
 	1850 1800 2150 1800
 Text Notes 4250 1450 0    50   ~ 0
-JP1: leave open until output of U3 is confirmed\nat 10.5V
+JP1: leave open until output of U3 is confirmed\nat 17V
 $Comp
 L Device:R_Small R?
@@
 AR Path="/630E4C46/641A8EE8" Ref="R?"  Part="1"
 F 0 "R36" H 4209 2871 50  0000 L CNN
-F 1 "1k" H 4209 2780 50  0000 L CNN
+F 1 "1500" H 4209 2780 50  0000 L CNN
 F 2 "Resistor_SMD:R_0805_2012Metric" H 4150 2825 50  0001 C CNN
 F 3 "~" H 4150 2825 50  0001 C CNN
@@
 P 8775 3775
 F 0 "C5" H 8867 3821 50  0000 L CNN
-F 1 "C_Small" H 8867 3730 50  0000 L CNN
+F 1 "100nF" H 8867 3730 50  0000 L CNN
 F 2 "Capacitor_SMD:C_1210_3225Metric_Pad1.33x2.70mm_HandSolder" H 8775 3775 50  0001 C CNN
 F 3 "~" H 8775 3775 50  0001 C CNN
@@
 P 9325 3775
 F 0 "C6" H 9417 3821 50  0000 L CNN
-F 1 "C_Small" H 9417 3730 50  0000 L CNN
+F 1 "100nF" H 9417 3730 50  0000 L CNN
 F 2 "Capacitor_SMD:C_1210_3225Metric_Pad1.33x2.70mm_HandSolder" H 9325 3775 50  0001 C CNN
 F 3 "~" H 9325 3775 50  0001 C CNN
